File: HVMeausrement.kicad_sch (KiCad schematic)
At the start: 12 parts, among them U7 AMC3336-Q1

Commit message: finished routing, sending to fab
Parts:
- C25: value 1nF -> (none); footprint Capacitor_SMD:C_0603_1608Metric -> (none)
- C26, C28: value 1uF -> (none); footprint Capacitor_SMD:C_0603_1608Metric -> (none)
- C27, C29, C32: value 100nF -> (none); footprint Capacitor_SMD:C_0603_1608Metric -> (none)
- R19, R22, R23: value 100k -> (none); footprint PD_HV_footprints:RESC1632X60N -> (none)
- R20: value 1k -> (none); footprint Resistor_SMD:R_0603_1608Metric -> (none)
- R21: value 4k7 -> (none); footprint Resistor_SMD:R_0603_1608Metric -> (none)
- U7: value AMC3336-Q1 -> (none); footprint Package_SO:SOIC-16W_7.5x10.3mm_P1.27mm -> (none)
Changed lines of the file:
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@@
       (effects (font (size 1.27 1.27)) (justify left))
     )
-    (property "Value" "100k" (id 1) (at 72.39 49.5299 0)
-      (effects (font (size 1.27 1.27)) (justify left))
-    )
-    (property "Footprint" "PD_HV_footprints:RESC1632X60N" (id 2) (at 68.072 48.26 90)
+    (property "Value" "" (id 1) (at 72.39 49.5299 0)
+      (effects (font (size 1.27 1.27)) (justify left))
+    )
+    (property "Footprint" "" (id 2) (at 68.072 48.26 90)
       (effects (font (size 1.27 1.27)) hide)
     )
@@
     (in_bom yes) (on_board yes) (fields_autoplaced)
     (property "Reference" "C26" (id 0) (at 100.33 39.37 90))
-    (property "Value" "1uF" (id 1) (at 100.33 41.91 90))
-    (property "Footprint" "Capacitor_SMD:C_0603_1608Metric" (id 2) (at 104.14 46.0248 0)
+    (property "Value" "" (id 1) (at 100.33 41.91 90))
+    (property "Footprint" "" (id 2) (at 104.14 46.0248 0)
       (effects (font (size 1.27 1.27)) hide)
     )
@@
       (effects (font (size 1.27 1.27)) (justify right))
     )
-    (property "Value" "1uF" (id 1) (at 168.91 73.6599 0)
+    (property "Value" "" (id 1) (at 168.91 73.6599 0)
       (effects (font (size 1.27 1.27)) (justify right))
     )
-    (property "Footprint" "Capacitor_SMD:C_0603_1608Metric" (id 2) (at 164.1348 68.58 0)
+    (property "Footprint" "" (id 2) (at 164.1348 68.58 0)
       (effects (font (size 1.27 1.27)) hide)
     )
@@
       (effects (font (size 1.27 1.27)) (justify left))
     )
-    (property "Value" "1k" (id 1) (at 72.39 77.4699 0)
-      (effects (font (size 1.27 1.27)) (justify left))
-    )
-    (property "Footprint" "Resistor_SMD:R_0603_1608Metric" (id 2) (at 68.072 76.2 90)
+    (property "Value" "" (id 1) (at 72.39 77.4699 0)
+      (effects (font (size 1.27 1.27)) (justify left))
+    )
+    (property "Footprint" "" (id 2) (at 68.072 76.2 90)
       (effects (font (size 1.27 1.27)) hide)
     )
@@
     (in_bom yes) (on_board yes) (fields_autoplaced)
     (property "Reference" "C27" (id 0) (at 100.33 59.69 90))
-    (property "Value" "100nF" (id 1) (at 100.33 62.23 90))
-    (property "Footprint" "Capacitor_SMD:C_0603_1608Metric" (id 2) (at 104.14 66.3448 0)
+    (property "Value" "" (id 1) (at 100.33 62.23 90))
+    (property "Footprint" "" (id 2) (at 104.14 66.3448 0)
       (effects (font (size 1.27 1.27)) hide)
     )
@@
       (effects (font (size 1.27 1.27)) (justify left))
     )
-    (property "Value" "100k" (id 1) (at 72.39 58.4199 0)
-      (effects (font (size 1.27 1.27)) (justify left))
-    )
-    (property "Footprint" "PD_HV_footprints:RESC1632X60N" (id 2) (at 68.072 57.15 90)
+    (property "Value" "" (id 1) (at 72.39 58.4199 0)
+      (effects (font (size 1.27 1.27)) (justify left))
+    )
+    (property "Footprint" "" (id 2) (at 68.072 57.15 90)
       (effects (font (size 1.27 1.27)) hide)
     )
@@
     (in_bom yes) (on_board yes) (fields_autoplaced)
     (property "Reference" "U7" (id 0) (at 132.08 39.37 0))
-    (property "Value" "AMC3336-Q1" (id 1) (at 132.08 41.91 0))
-    (property "Footprint" "Package_SO:SOIC-16W_7.5x10.3mm_P1.27mm" (id 2) (at 132.08 46.99 0)
+    (property "Value" "" (id 1) (at 132.08 41.91 0))
+    (property "Footprint" "" (id 2) (at 132.08 46.99 0)
       (effects (font (size 1.27 1.27)) hide)
     )
@@
       (effects (font (size 1.27 1.27)) (justify left))
     )
-    (property "Value" "4k7" (id 1) (at 156.21 40.6399 0)
-      (effects (font (size 1.27 1.27)) (justify left))
-    )
-    (property "Footprint" "Resistor_SMD:R_0603_1608Metric" (id 2) (at 151.892 39.37 90)
+    (property "Value" "" (id 1) (at 156.21 40.6399 0)
+      (effects (font (size 1.27 1.27)) (justify left))
+    )
+    (property "Footprint" "" (id 2) (at 151.892 39.37 90)
       (effects (font (size 1.27 1.27)) hide)
     )
@@
       (effects (font (size 1.27 1.27)) (justify left))
     )
-    (property "Value" "1nF" (id 1) (at 87.63 77.4699 0)
-      (effects (font (size 1.27 1.27)) (justify left))
-    )
-    (property "Footprint" "Capacitor_SMD:C_0603_1608Metric" (id 2) (at 84.7852 80.01 0)
+    (property "Value" "" (id 1) (at 87.63 77.4699 0)
+      (effects (font (size 1.27 1.27)) (justify left))
+    )
+    (property "Footprint" "" (id 2) (at 84.7852 80.01 0)
       (effects (font (size 1.27 1.27)) hide)
     )
@@
     (in_bom yes) (on_board yes)
     (property "Reference" "C32" (id 0) (at 81.28 48.26 90))
-    (property "Value" "100nF" (id 1) (at 86.36 48.26 90))
-    (property "Footprint" "Capacitor_SMD:C_0603_1608Metric" (id 2) (at 92.71 51.1048 0)
+    (property "Value" "" (id 1) (at 86.36 48.26 90))
+    (property "Footprint" "" (id 2) (at 92.71 51.1048 0)
       (effects (font (size 1.27 1.27)) hide)
     )
@@
       (effects (font (size 1.27 1.27)) (justify right))
     )
-    (property "Value" "100nF" (id 1) (at 179.07 73.6599 0)
+    (property "Value" "" (id 1) (at 179.07 73.6599 0)
       (effects (font (size 1.27 1.27)) (justify right))
     )
-    (property "Footprint" "Capacitor_SMD:C_0603_1608Metric" (id 2) (at 174.2948 68.58 0)
+    (property "Footprint" "" (id 2) (at 174.2948 68.58 0)
       (effects (font (size 1.27 1.27)) hide)
     )
@@
       (effects (font (size 1.27 1.27)) (justify left))
     )
-    (property "Value" "100k" (id 1) (at 72.39 67.3099 0)
-      (effects (font (size 1.27 1.27)) (justify left))
-    )
-    (property "Footprint" "PD_HV_footprints:RESC1632X60N" (id 2) (at 68.072 66.04 90)
-      (effects (font (size 1.27 1.27)) hide)
-    )
+    (property "Value" "" (id 1) (at 72.39 67.3099 0)
+      (effects (font (size 1.27 1.27)) (justify left))
+    )
+    (property "Footprint" "" (id 2) (at 68.072 66.04 90)
+      (effects (font (size 1.27 1.27)) hide)
+    )
