File: USBPD_IN.kicad_sch (KiCad schematic)
At the start: 13 parts, among them J1 USB_C_Receptacle, Q2 AON7410, Q3 AO3400A, U3 IP2721

Commit message: finished routing, sending to fab
Parts:
- added TP_20VPD1, TP_3V3, TP_VBUS1, TP_VBUSG1: (no value), symbol Connector:TestPoint
- C10: value 22uF -> (none); footprint Capacitor_SMD:C_0603_1608Metric -> (none)
- C7: value 1uF -> (none); footprint Capacitor_SMD:C_0603_1608Metric -> (none)
- C8, C9: value 10uF -> (none); footprint Capacitor_SMD:C_0805_2012Metric -> (none)
- D1: value ESDA6V1BC6 -> (none); footprint Package_TO_SOT_SMD:SOT-23-6 -> (none)
- J1: value USB_C_Receptacle -> (none); footprint Connector_USB:USB_C_Receptacle_JAE_DX07S016JA1R1500 -> (none)
- MOD1: value K7803JT-500R3-LB -> (none); footprint PD_HV_footprints:MORNSUN_K7803JT-500R3-LB -> (none)
- Q2: value AON7410 -> (none); footprint PD_HV_footprints:DFN3X3A_8L_EPA1_P_AOS -> (none)
- Q3: value AO3400A -> (none); footprint Package_TO_SOT_SMD:SOT-23 -> (none)
- R10: value 100k -> (none); footprint Resistor_SMD:R_0603_1608Metric -> (none)
- R8, R9: value 5.1k -> (none); footprint Resistor_SMD:R_0603_1608Metric -> (none)
- U3: value IP2721 -> (none); footprint Package_SO:TSSOP-16_4.4x5mm_P0.65mm -> (none)
Connections:
- net +20V_USBPD: now also TP_20VPD1.1
- net +3.3V: now also TP_3V3.1
- net VBUS: now also TP_VBUS1.1
- net VBUSG: now also TP_VBUSG1.1
