File: rp2040.kicad_sch (KiCad schematic)
At the start: 21 parts, among them SW1 SW_SPST, SW2 SW_SPST, U5 RP2040, U6 W25Q128JVS, Y1 Crystal

Commit message: finished routing, sending to fab
Parts:
- added J4: (no value), symbol Connector:Conn_01x04_Male
- added R24, R25: (no value), symbol Device:R
- added SW4: (no value), symbol PDHV_sym:MOM-OFF-MOM
- added SW5: (no value), symbol PDHV_sym:SW_SPDT
- added TP_3V3_MIC1, TP_CLKIN1, TP_DEC1, TP_DIAG1, TP_DOUT1, TP_GND1, TP_GND2, TP_INC1, TP_ONOFF1, TP_SCLK1, TP_SD1, TP_SD2, TP_SD3, TP_SDO1, TP_SS1: (no value), symbol Connector:TestPoint
- C11, C14: value 27p -> (none); footprint Capacitor_SMD:C_0603_1608Metric -> (none)
- C12, C21: value 1uF -> (none); footprint Capacitor_SMD:C_0603_1608Metric -> (none)
- C13, C15, C17, C18, C19, C20, C22, C23, C24: value 100nF -> (none); footprint Capacitor_SMD:C_0603_1608Metric -> (none)
- R16, R17: value 1k -> (none); footprint Resistor_SMD:R_0603_1608Metric -> (none)
- R18: value 10k -> (none); footprint Resistor_SMD:R_0603_1608Metric -> (none)
- SW1, SW2: value SW_SPST -> (none); footprint Button_Switch_SMD:SW_SPST_PTS645 -> (none)
- U5: value RP2040 -> (none); footprint RP2040:QFN40P700X700X90-57N -> (none)
- U6: value W25Q128JVS -> (none); footprint Package_SO:SOIC-8_5.23x5.23mm_P1.27mm -> (none)
- Y1: value Crystal -> (none); footprint PD_HV_footprints:ABLS-2SMD-XTAL -> (none)
Connections:
- net +3.3V: now also J4.4 (Pin_4), R24.1, R25.1, TP_3V3_MIC1.1
- net GND: now also J4.1 (Pin_1), SW4.2, SW5.2, TP_GND1.1, TP_GND2.1
- net QSPI_SCLK: now also TP_SCLK1.1
- net QSPI_SD0: now also TP_SDO1.1
- net QSPI_SD1: now also TP_SD1.1
- net QSPI_SD2: now also TP_SD2.1
- net QSPI_SD3: now also TP_SD3.1
- net QSPI_SS: now also TP_SS1.1
- net SCL_I2C0: now also J4.2 (Pin_2), R25.2
- net SDA_I2C0: now also J4.3 (Pin_3), R24.2
- net ONOFF: now reaches U5.12 (GPIO9)
- net ONOFF: now also SW5.3, TP_ONOFF1.1
- net INC: now reaches U5.13 (GPIO10)
- net INC: now also SW4.3, TP_INC1.1
- net DEC: now reaches U5.14 (GPIO11)
- net DEC: now also SW4.1, TP_DEC1.1
- net CLKIN: now reaches U5.38 (GPIO26/ADC0)
- net CLKIN: now also TP_CLKIN1.1
- net DIAG: now reaches U5.39 (GPIO27/ADC1)
- net DIAG: now also TP_DIAG1.1
- net DOUT: now reaches U5.40 (GPIO28/ADC2)
- net DOUT: now also TP_DOUT1.1
Other:
- note removed: "PULLUPS ON HV SCHEMATIC"
- moved on the sheet: SW1, SW2
